File: LinHT-rf-amp.kicad_pcb (KiCad board)
At the start: 4 copper layers, 40 x 20 mm, 27 parts, among them J1 SIGNALS, J2 INPUT, J3 OUTPUT, U1 GRF5604

Commit message: silkscreen update
frequency range starts at 397 MHz
Other:
- board text added: "LinHT 397-470 MHz Power Amplifier GRF5604 6 Watt"
- board text removed: "LinHT 390-470 MHz Power Amplifier GRF5604 6 Watt"
Changed lines of the file:
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@@
 		)
 	)
-	(gr_text "LinHT \n390-470 MHz Power Amplifier\nGRF5604 6 Watt"
+	(gr_text "LinHT \n397-470 MHz Power Amplifier\nGRF5604 6 Watt"
 		(at 154.37 92.375 0)
 		(layer "B.SilkS")
